File: pcb/StarDuino2812/StarDuino.sch (KiCad schematic (older format))
At the start: 91 parts, among them J1 Screw_Terminal_01x02, J2 Conn_01x03_Male, J3 Conn_01x01_Male, Q1 IRLML6401, U1 ATmega328P-AU, Y1 16M

Commit message: Add ISP to StarDuino
Parts:
- added J4, J5, J6: Conn_01x01_Male, Connector_PinHeader_2.54mm:PinHeader_1x01_P2.54mm_Vertical, symbol Connector:Conn_01x01_Male
Connections:
- net MOSI: now reaches U1.15 (PB3)
- net MOSI: now also J4.1 (Pin_1)
- net MISO: now reaches U1.16 (PB4)
- net MISO: now also J5.1 (Pin_1)
- net SCK: now reaches U1.17 (PB5)
- net SCK: now also J6.1 (Pin_1)
- no-connect marks 26 -> 23
Changed lines of the file:
@@
 NoConn ~ 2950 4350
 NoConn ~ 2950 4450
-NoConn ~ 2950 4550
-NoConn ~ 2950 4650
-NoConn ~ 2950 4750
 NoConn ~ 2950 5150
 NoConn ~ 2950 5350
@@
 	1    0    0    -1
 $EndComp
+Text Label 2950 4650 0    50   ~ 0
+MISO
+Text Label 2950 4750 0    50   ~ 0
+SCK
+Text Label 2950 4550 0    50   ~ 0
+MOSI
+$Comp
+L Connector:Conn_01x01_Male J6
+U 1 1 61B3A953
+P 3150 4750
+F 0 "J6" H 3122 4774 50  0000 R CNN
+F 1 "Conn_01x01_Male" H 3000 4775 50  0000 R CNN
+F 2 "Connector_PinHeader_2.54mm:PinHeader_1x01_P2.54mm_Vertical" H 3150 4750 50  0001 C CNN
+F 3 "~" H 3150 4750 50  0001 C CNN
+	1    3150 4750
+	-1   0    0    -1
+$EndComp
+$Comp
+L Connector:Conn_01x01_Male J5
+U 1 1 61B6491A
+P 3150 4650
+F 0 "J5" H 3122 4674 50  0000 R CNN
+F 1 "Conn_01x01_Male" H 3000 4675 50  0000 R CNN
+F 2 "Connector_PinHeader_2.54mm:PinHeader_1x01_P2.54mm_Vertical" H 3150 4650 50  0001 C CNN
+F 3 "~" H 3150 4650 50  0001 C CNN
+	1    3150 4650
+	-1   0    0    -1
+$EndComp
+$Comp
+L Connector:Conn_01x01_Male J4
+U 1 1 61B64C04
+P 3150 4550
+F 0 "J4" H 3122 4574 50  0000 R CNN
+F 1 "Conn_01x01_Male" H 3000 4575 50  0000 R CNN
+F 2 "Connector_PinHeader_2.54mm:PinHeader_1x01_P2.54mm_Vertical" H 3150 4550 50  0001 C CNN
+F 3 "~" H 3150 4550 50  0001 C CNN
+	1    3150 4550
+	-1   0    0    -1
+$EndComp
 $EndSCHEMATC
